File: mixlib-kicad.kicad_sch (KiCad schematic)
At the start: 0 parts

Commit message: feat: various improvements, components and simulation scripts
Parts:
- added R1, R11, R12, R13, R2: 10k, symbol Device:R_Small
- added U1, U2: MCP6401, Package_TO_SOT_SMD:SOT-353_SC-70-5, symbol mixlib-analog-opamp:MCP6401
- added V1, V2: 5, symbol Simulation_SPICE:VDC
Connections:
- new net: R12.1, R13.2, U2.4 (-)
- new net: R11.1, R12.2, U1.3 (+)
- new net GND: R1.1, R13.1, R2.1, U1.2 (V-), U2.2 (V-), V1.2, V2.2
- new net VCC: R11.2, U1.5 (V+), U2.5 (V+), V2.1
- new net VG: U1.4 (-), U2.3 (+), V1.1
- new net VOUT1: R2.2, U1.1
- new net VOUT2: R1.2, U2.1
