File: mixlib-kicad.kicad_sch (KiCad schematic)
At the start: 52 parts, among them Q1 MMBT5551L, Q2 MMBT5551L, Q3 PMD3001D, Q4 PBSS4160DS, Q6 PBSS4160DPN, U1 ADA4522-4, U2 MCP6404, U3 ADA4522-2, U4 LM4040DBZ-10, U5 TPS5430DDA, U6 TJ-S1615CY6TGLCCYRGY-A5, U7 CH32V006K8U6

Commit message: feat(connector-general): add barrel jack connector with 3D model
Parts:
- added U8: TXS0102DQE, mixlib-vendor-ti:vendor-ti-DQE0008A, symbol mixlib-ic-logic:TXS0102DQE
- added U9: TXS0102DQE, Package_SON:X2SON-8_1.4x1mm_P0.35mm, symbol Logic_LevelTranslator:TXS0102DQE
Changed lines of the file:
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@@
 	)
 	(symbol
+		(lib_id "mixlib-ic-logic:TXS0102DQE")
+		(at 226.06 33.02 0)
+		(unit 1)
+		(body_style 1)
+		(exclude_from_sim no)
+		(in_bom yes)
+		(on_board yes)
+		(in_pos_files yes)
+		(dnp no)
+		(fields_autoplaced yes)
+		(property "Reference" "U8"
+			(at 228.2033 45.72 0)
+			(show_name no)
+			(do_not_autoplace no)
+			(effects
+				(font
+					(size 1.27 1.27)
+				)
+				(justify left)
+			)
+		)
+		(property "Value" "TXS0102DQE"
+			(at 228.2033 48.26 0)
+			(show_name no)
+			(do_not_autoplace no)
+			(effects
+				(font
+					(size 1.27 1.27)
+				)
+				(justify left)
+			)
+		)
+		(property "Footprint" "mixlib-vendor-ti:vendor-ti-DQE0008A"
+			(at 226.06 46.99 0)
+			(hide yes)
+			(show_name no)
+			(do_not_autoplace no)
+			(effects
+				(font
+					(size 1.27 1.27)
+				)
+			)
+		)
+		(property "Datasheet" "http://www.ti.com/lit/gpn/txs0102"
+			(at 226.06 33.528 0)
+			(hide yes)
+			(show_name no)
+			(do_not_autoplace no)
+			(effects
+				(font
+					(size 1.27 1.27)
+				)
+			)
+		)
+		(property "Description" "2-Bit Bidirectional Voltage-Level Shifter for Open-Drain and Push-Pull Application, X2SON-8"
+			(at 226.06 33.02 0)
+			(hide yes)
+			(show_name no)
+			(do_not_autoplace no)
+			(effects
+				(font
+					(size 1.27 1.27)
+				)
+			)
+		)
+		(pin "7"
+		)
+		(pin "8"
+		)
+		(pin "2"
+		)
+		(pin "4"
+		)
+		(pin "1"
+		)
+		(pin "3"
+		)
+		(pin "5"
+		)
+		(pin "6"
+		)
+		(instances
+			(project "mixlib-kicad"
+				(path "/addedff5-7d4f-4971-a0ac-6e5a34b85b52"
+					(reference "U8")
+					(unit 1)
+				)
+			)
+		)
+	)
+	(symbol
 		(lib_id "Simulation_SPICE:VDC")
 		(at 255.27 115.57 0)
@@
 					(unit 1)
 				)
+			)
+		)
+	)
+	(symbol
+		(lib_id "Logic_LevelTranslator:TXS0102DQE")
+		(at 257.81 31.75 0)
+		(unit 1)
+		(body_style 1)
+		(exclude_from_sim no)
+		(in_bom yes)
+		(on_board yes)
+		(in_pos_files yes)
+		(dnp no)
+		(fields_autoplaced yes)
+		(property "Reference" "U9"
+			(at 259.9533 44.45 0)
+			(show_name no)
+			(do_not_autoplace no)
+			(effects
+				(font
+					(size 1.27 1.27)
+				)
+				(justify left)
+			)
+		)
+		(property "Value" "TXS0102DQE"
+			(at 259.9533 46.99 0)
+			(show_name no)
+			(do_not_autoplace no)
+			(effects
+				(font
+					(size 1.27 1.27)
+				)
+				(justify left)
+			)
+		)
+		(property "Footprint" "Package_SON:X2SON-8_1.4x1mm_P0.35mm"
+			(at 257.81 45.72 0)
+			(hide yes)
+			(show_name no)
+			(do_not_autoplace no)
+			(effects
+				(font
+					(size 1.27 1.27)
+				)
+			)
+		)
+		(property "Datasheet" "http://www.ti.com/lit/gpn/txs0102"
+			(at 257.81 32.258 0)
+			(hide yes)
+			(show_name no)
+			(do_not_autoplace no)
+			(effects
+				(font
+					(size 1.27 1.27)
+				)
+			)
+		)
+		(property "Description" "2-Bit Bidirectional Voltage-Level Shifter for Open-Drain and Push-Pull Application, X2SON-8"
+			(at 257.81 31.75 0)
+			(hide yes)
+			(show_name no)
+			(do_not_autoplace no)
+			(effects
+				(font
+					(size 1.27 1.27)
+				)
+			)
+		)
+		(pin "6"
+		)
+		(pin "4"
+		)
+		(pin "5"
+		)
+		(pin "1"
+		)
+		(pin "7"
+		)
+		(pin "8"
+		)
+		(pin "3"
+		)
+		(pin "2"
+		)
+		(instances
+			(project "mixlib-kicad"
+				(path "/addedff5-7d4f-4971-a0ac-6e5a34b85b52"
+					(reference "U9")
+					(unit 1)
+				)

Commit message: feat(discrete-resistor): add small-symbol 4-pin resistor pack
Parts:
- removed Q1, Q2: MMBT5551L, Package_TO_SOT_SMD:SOT-23, symbol mixlib-discrete-npn:MMBT5551L
- removed Q3: PMD3001D, mixlib-generic-sot:SC-74_SOT-457_NEX, symbol mixlib-discrete-npnpnp:PMD3001D
- removed Q4: PBSS4160DS, mixlib-generic-sot:SC-74_SOT-457_NEX, symbol mixlib-discrete-npn:PBSS4160DS
- removed Q6: PBSS4160DPN, mixlib-generic-sot:SC-74_SOT-457_NEX, symbol mixlib-discrete-npnpnp:PBSS4160DPN
- removed R10: 560, symbol Device:R_Small
- removed R11, R19, R20, R21, R24, R25, R7, R8: 10k, symbol Device:R_Small
- removed R15: 4.7k, symbol Device:R_Small
- removed R22: 200k, symbol Device:R_Small
- removed R23: 470, symbol Device:R_Small
- removed R26, R27, R28: R_Small, symbol Device:R_Small
- removed S1, S2: SWITCH, symbol Simulation_SPICE:SWITCH
- removed U1: ADA4522-4, symbol mixlib-analog-opamp:ADA4522-4
- removed U2: MCP6404, Package_SO:SOIC-14_3.9x8.7mm_P1.27mm, symbol mixlib-analog-opamp:MCP6404
- removed U3: ADA4522-2, symbol mixlib-analog-opamp:ADA4522-2
- removed U4: LM4040DBZ-10, Package_TO_SOT_SMD:SOT-23, symbol Reference_Voltage:LM4040DBZ-10
- removed U5: TPS5430DDA, Package_SO:TI_SO-PowerPAD-8_ThermalVias, symbol mixlib-pmic-vreg:TPS5430DDA
- removed U6: TJ-S1615CY6TGLCCYRGY-A5, mixlib-discrete-led:LED-3_RGB-0603_1615Metric, symbol mixlib-discrete-led:TJ-S1615CY6TGLCCYRGY-A5
- removed U7: CH32V006K8U6, Package_DFN_QFN:QFN-32-1EP_4x4mm_P0.4mm_EP2.9x2.9mm, symbol mixlib-ic-mcu:CH32V006K8U6
- removed U8: TXS0102DQE, mixlib-vendor-ti:vendor-ti-DQE0008A, symbol mixlib-ic-logic:TXS0102DQE
- removed U9: TXS0102DQE, Package_SON:X2SON-8_1.4x1mm_P0.35mm, symbol Logic_LevelTranslator:TXS0102DQE
- removed V1: 50, symbol Simulation_SPICE:VDC
- removed V10: VPWM, symbol mixlib-sim-vsource:VPWM
- removed V3, V8: VSIN, symbol Simulation_SPICE:VSIN
- removed V6: 5, symbol Simulation_SPICE:VDC
- removed V7: -5, symbol Simulation_SPICE:VDC
- added D1, D3, D8: 1N4148WS, Diode_SMD:D_SOD-323, symbol mixlib-discrete-diode:1N4148WS
- added D2, D4: BZT52C15, Diode_SMD:D_SOD-123, symbol mixlib-discrete-zener:BZT52Cxx
- added D6: SS36, Diode_SMD:D_SMA, symbol mixlib-discrete-schottkydiode:SS36
- added D7: BZT52C3V3, Diode_SMD:D_SOD-123, symbol mixlib-discrete-zener:BZT52Cxx
- added Q1, Q3: AO3401A, Package_TO_SOT_SMD:SOT-23, symbol mixlib-discrete-mosfet:AO3401A
- added Q2: BSS138PS, mixlib-generic-sot:SOT-363_SC-70-6, symbol mixlib-discrete-mosfet:BSS138PS
- added V3: 5, symbol Simulation_SPICE:VDC
- C1: value 2.2n -> 1u
- R1, R12, R13, R18, R3: value 10k -> 1M
- R14, R2, R4: value 10k -> 1k
- R16: value 10k -> 470k
- R17: value 200k -> 1M
- R6: value 10k -> 4.7k
- R9: value 1.5k -> 10k
- V2: value 50 -> 3.3
- V4: value 2.5 -> 20
- V5: value 45 -> 24
Connections:
- net VDRIVER_VSS is gone; now on net GND: C1.2
- net VOUT_BOT is gone; now on an unnamed net: R1.2
- net VREF_TOP is gone; now on net GND: R12.2
- net VSIN_CMP_TOP is gone; now on net GND: R16.2, R6.2
- net VSIN_OUT2 is gone; now on an unnamed net: R17.1
- net VSIN_VREF is gone; now on net +24V: V5.1
- net GND: now also R13.2, R14.2, R17.2, R2.2, R4.2, D1.1 (K), D3.2 (A), Q2.4 (S), V3.2; no longer R13.1
- net +5V: now reaches C1.1
- net +5V: now also R13.1, R5.1, D6.2 (A), D7.1 (K), D8.2 (A), V3.1
- net at R16.1: now also D4.2 (A), D8.1 (K), Q3.1 (G)
- net +3V3: now reaches R3.1
- net +3V3: now also R6.1, R9.1, V2.1
- net at R5.2: now also D3.1 (K); no longer R9.1
- net at R9.2: now also Q2.3 (D); no longer R6.1
- net at R18.1: now also D7.2 (A); no longer R4.2
- net +24V: now reaches R1.1
- net +24V: now also D2.1 (K), Q1.2 (S)
- removed net VCC: R14.2, R2.2, V2.1
- net VOUT: no longer names the net of R2.1
- net VOUT: now also D2.2 (A), Q1.1 (G)
- net VOUT_TOP: no longer names the net of R3.2
- net VOUT_TOP: now also D1.2 (A)
- net VREF: no longer names the net of R4.1
- net VREF: now also Q1.3 (D); no longer V4.1
- net VREFZ: no longer names the net of R14.1
- net VREFZ: now also D4.1 (K), D6.1 (K), Q3.2 (S)
- net VREF_BOT: no longer names the net of R12.1
- net VREF_BOT: now also Q3.3 (D); no longer R13.2
- net VSIN_CMP_BOT: no longer names the net of R18.2
- net VSIN_CMP_BOT: now also Q2.5 (G); no longer R5.1
- new net +20V: V4.1
